File: sensor-water.sch (KiCad schematic (older format))
At the start: 86 parts, among them IC1 STM8S003F3P, P1 CONN_01X04, P2 CONN_01X06, P3 CONN_01X03, P4 CONN_01X04, Q1 C1815, Q2 C1815, U1 LM358D, U10 -6V5, U11 6V5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

Commit message: initial README.md
Parts:
- removed C1: 100nF/10V, symbol CAP
- removed C11, C13, C14, C15, C16: 100nF/50V, symbol CAP
- removed C18: 1u/50V, symbol CP1
- removed C19: 1uF, symbol CAP
- removed C2: 10uF/10V, symbol CAP
- removed C20: 4.7uF, symbol CAP
- removed C3: 100uF/10V, symbol CAP
- removed IC1: STM8S003F3P, TSSOP-20, symbol STM8S003F3P
- removed P1, P4: CONN_01X04, symbol CONN_01X04
- removed P3: CONN_01X03, symbol CONN_01X03
- removed R22: 10K,5%, symbol R
- removed R23: R, symbol R
- removed U10, U14, U17, U3, U5, U8, U? (x2): -6V5, symbol -6V5
- removed U11, U13, U15, U2, U6, U7, U? (x4): 6V5, symbol 6V5
- removed U18: LP2985LV, symbol LP2985LV
- added C? (x2): 100nF/10V, symbol CAP
- added C?: 10nF/10V, symbol CAP
- added C? (x5): 100nF/50V, symbol CAP
- added C?: 1uF, symbol CAP
- added C?: 1u/50V, symbol CP1
- added C?: 4.7uF, symbol CAP
- added IC?: STM8S003F3P-RESCUE-sensor-water, TSSOP-20, symbol STM8S003F3P-RESCUE-sensor-water
- added P?: CONN_01X03, symbol CONN_01X03
- added P? (x2): CONN_01X04, symbol CONN_01X04
- added R?: 10K.5%, symbol R
- added R?: 4K7, symbol R
- added U? (x8): -6V5, symbol -6V5
- added U?: LP2985LV, symbol LP2985LV
- added _? (x10): 6V5, symbol 6V5
- R10, R9: value R -> 10K
- R11, R12: value R -> 2.2K
- U1, U9: symbol LM358 -> LM358-RESCUE-sensor-water
Connections:
- net labels added: NRST, SEMSOR, SENSOR, SWIM
- wire segments 161 -> 188
- no-connect marks 3 -> 10
Other:
- moved on the sheet: P2

Commit message: initial README.md
Parts:
- removed P2: CONN_01X06, symbol CONN_01X06
- removed U?: -6V5, symbol -6V5
- removed _? (x10): 6V5, symbol 6V5
- added P2, P5, P6, P7, P8, P9: CONN_01X01, symbol CONN_01X01
- U12: renamed from U?; symbol LP2985LV -> LP2985LV-RESCUE-sensor-water
- gave numbers to parts that had none: 24
Connections:
- net SEMSOR is gone; now on net SENSOR: P4.2 (P2), R23.1
- net CON-IN: now also P8.1 (P1)
- net CON-OUT: now also P9.1 (P1)
- net COND-OFF: now also IC1.15 ([TIM2_CH1]SPI_SCK/PC5)
- net COND-PWM: now also Q2.2 (C), R9.1
- net GND: now also C19.2
- net W-1: now also P5.1 (P1)
- net W-2: now also P6.1 (P1)
- net W-3: now also P7.1 (P1)
- net WATER-ON: now also IC1.13 ([TIM1_CH1N]TIM1_CH3/PC3)
- net WATER-OUT: now also D3.1 (K), D4.2 (A), R14.2, P2.1 (P1)
- net WATER-PWM: now also Q1.2 (C), R10.1
- net at U16.11 (-): now also U16.11 (-), U16.11 (-), U16.4 (+)
- net at U16.4 (+): now also U11.~ (-6V5), U16.11 (-), U16.4 (+), U16.4 (+)
- net at C4.2, C6.2, C8.2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: now also C5.2
- no-connect marks 10 -> 8
Other:
- note added: "INPUT"
- note added: "OUTPUT"
- moved on the sheet: C1, C11, C13, C14, C15, C16, C2, C3, C4, C5, C6, C8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
