File: _saved_sensor-water.sch (KiCad schematic (older format))
At the start: 75 parts, among them IC1 STM8S003F3P-RESCUE-sensor-wat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, P1 CONN_01X04, P2 CONN_01X01, P3 CONN_01X04, P4 CONN_01X03, P5 CONN_01X01, P6 CONN_01X01, P7 CONN_01X01, P8 CONN_01X01, P9 CONN_01X01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

Commit message: initial kicad-sensor-water
Parts:
- removed C1: 100uF/16V-phancuc, mylib:C_2920, symbol CAP
- removed C11, C13: 100nF/50V, mylib:C_2920, symbol CAP
- removed C18: 1u/50V, Capacitors_SMD:C_0805, symbol CP1
- removed C3: 100uF/16V-phan cuc, mylib:C_2920, symbol CAP
- removed IC1: STM8S003F3P-RESCUE-sensor-water-Stm32f030f4p6, Housings_SOIC:SOIC-20_7.5x12.8mm_Pitch1.27mm, symbol STM8S003F3P-RESCUE-sensor-water
- removed P4: CONN_01X03, Pin_Headers:Pin_Header_Angled_1x03, symbol CONN_01X03
- added C1, C3: 100uF/16V, Capacitors_SMD:C_1206_HandSoldering, symbol CP1
- added IC1: STM32F030F4P6, mylib:STM32F030F4P6, symbol STM32F030F4P6
- added R26: 10K, Resistors_SMD:R_0805_HandSoldering, symbol R
- added U2: DS18B20, TO_SOT_Packages_THT:TO-92_Horizontal2_Inline_Narrow_Oval, symbol DS18B20
- C10, C12, C14, C15, C16, C6, C7, C8, C9: footprint mylib:C_2920 -> Capacitors_SMD:C_0805_HandSoldering
- C2: value 10uF/16V-1206 -> 10uF/16V; footprint Capacitors_SMD:C_0805_HandSoldering -> Capacitors_SMD:C_1206_HandSoldering
- C4, C5: value 100nF/50V -> 100nF/16V; footprint mylib:C_2920 -> Capacitors_SMD:C_0805_HandSoldering
- U1, U9: footprint Housings_SOIC:SOIC-8-1EP_3.9x4.9mm_Pitch1.27mm -> Housings_SOIC:SOIC-8_3.9x4.9mm_Pitch1.27mm
Connections:
- net labels added: +12V, +3.3V, SWCLK, SWDIO
- net labels removed: +12VA, +9VA, -9VA, SWIM, VCC
- wire segments 198 -> 197
- no-connect marks 8 -> 6
Other:
- moved on the sheet: C14, C15, C16, C19, C20, C6, C8, C9, R22, U12
